File: pcb/ES_Daisy_Seed2_DFM_EVAL_PEDAL_Rev5_3.kicad_sch (KiCad schematic)
At the start: 61 parts, among them U1 MCP6002-xSN, U10 OPA1652, U3 OPA1652, U9 OPA1652

Commit message: everything's on the board.
Parts:
- removed C18, C58: 10UF, PANASONIC_B, symbol Seed3-Pedal-DevKit-Converted-eagle-import:C-EU-POL_B
- removed C19: 100NF, C0402_29888544, symbol Seed3-Pedal-DevKit-Converted-eagle-import:Electrosmith-Passives_C-EUC0402
- removed C40: 100UF DNI, PANASONIC_D, symbol Seed3-Pedal-DevKit-Converted-eagle-import:C-EU-POL_D
- removed FB6: FERRITE_BEAD_0603, WUERTH-ELEKTRONIK_0603, symbol Seed3-Pedal-DevKit-Converted-eagle-import:FERRITE_BEAD_0603
- added C17, C25: 100NF, Capacitor_SMD:C_0603_1608Metric, symbol Seed3-Pedal-DevKit-Converted-eagle-import:Electrosmith-Passives_C-EUC0402
- added unit 3 of U3
- C10, C29, C3, C35, C42, C48, C6, C7: footprint (none) -> Capacitor_SMD:CP_Elec_4x5.8
- C11, C28, C30, C32, C38, C5, C8, C9: footprint (none) -> Capacitor_SMD:C_0603_1608Metric
- C12, C37: value C -> 33NF; footprint (none) -> Capacitor_SMD:C_0603_1608Metric
- C2, C4: footprint C0402_29888544 -> Capacitor_SMD:C_0603_1608Metric
- C33: footprint C0402 -> Capacitor_SMD:C_0603_1608Metric
- C39: footprint PANASONIC_D -> Capacitor_SMD:CP_Elec_6.3x7.7; symbol Seed3-Pedal-DevKit-Converted-eagle-import:C-EU-POL_D -> Device:C_Polarized_US
- C46, C55: footprint C0603 -> Capacitor_SMD:C_0603_1608Metric
- R11, R12, R13, R14, R15, R16, R20, R21, R22, R26, R27, R58, R69, R7, R70, R71, R72, R74, R75, R76, R77, R8: footprint (none) -> Resistor_SMD:R_0603_1608Metric
- R17, R18, R5, R60: footprint R0603 -> Resistor_SMD:R_0603_1608Metric
- R19: value 1M DNI -> 10K; footprint R0603 -> Resistor_SMD:R_0603_1608Metric
- R56: value 0R -> 10K; footprint R0603 -> Resistor_SMD:R_0603_1608Metric
- U1, U10, U3, U9: footprint (none) -> Package_SO:SOIC-8_5.275x5.275mm_P1.27mm
Connections:
- net AREF_+2V5 is gone; now on net AREF_AUDIO_IN_BIAS: R5.1, U1.1, U1.2 (-)
- net AUDIO_BUFF_LEFT: no longer C7.2
- net AUDIO_DSP_LEFT: no longer C6.1, R14.1
- net CODEC_IN_L: no longer C12.2, R27.1
- net CODEC_OUT_L: no longer C3.2
- net GND: now also C39.2, U10.4 (V-), U9.4 (V-), C17.2, C25.2, U3.4 (V-); no longer C39.- (NEG)
- net +9V_A: now reaches U9.8 (V+)
- net +9V_A: now also C4.1, U10.8 (V+), C17.1, C25.1, U3.8 (V+)
- net +2V5_PRE: no longer names the net of C33.1, C55.1, R19.1, R56.2, U1.3 (+)
- net +2V5_PRE: now also C39.1; no longer C39.+ (POS)
- net +5V renamed +5V_A
- net +5V_A: now also C2.1, U1.8 (V+)
- net AREF_2v5_PRE renamed +3V3_A
- removed net CODEC_VCC: C2.1, C4.1, U1.8 (V+)
- new net AUDIO_BUFF_RIGHT: C7.2
- new net AUDIO_DSP_RIGHT: C6.1, R14.1
- new net CODEC_IN_R: C12.2, R27.1
- new net CODEC_OUT_R: C3.2
Other:
- note added: "--- Identical circuits for right audio channel ---"
- note added: "1.67V ref for audio bias"
- note added: "Fc = 1.5MHz This can be tested for removal"
- note added: "G = 1.6 (ideal 1.704) Fc = 66.3kHz"
- note added: "HPF = 0.15Hz"
- note added: "LPF Fc = 48kHz HPF Fc = 3Hz Gain pre-atten down to AK4558 levels G=0.58"
- note added: "prior stage RC filter could potentially be removed, and gain could happen here? Fc = 58.946kHz"
- note removed: "Audio Power"
- note removed: "Fc = 48kHz Gain pre-atten down to AK4558 levels G=0.58"
- note removed: "Very big cutoff Can probably remove"
- note removed: "prior stage RC filter could potentially be removed, and gain could happen here?"
- moved on the sheet: C2, R5, U10C, U1A, U1C, U9C
