File: pcb/ES_Daisy_Seed2_DFM_EVAL_PEDAL_Rev5_4.kicad_sch (KiCad schematic)
At the start: 30 parts, among them J7 GUITAR_DC_JACK, U4 LM4040DBZ-2.5, U8 LD1117-5V

Commit message: everything's on the board.
Parts:
- removed C17: 100NF, C0402, symbol Seed3-Pedal-DevKit-Converted-eagle-import:Electrosmith-Passives_C-EUC0402
- removed J7: GUITAR_DC_JACK, WQP-DC0500, symbol Seed3-Pedal-DevKit-Converted-eagle-import:GUITAR_DC_JACK
- removed R6: 2K, R0603, symbol Seed3-Pedal-DevKit-Converted-eagle-import:Electrosmith-Passives_R-US_R0603
- removed U4: LM4040DBZ-2.5, Package_TO_SOT_SMD:SOT-23, symbol Reference_Voltage:LM4040DBZ-2.5
- added C18, C19: 10UF, Capacitor_SMD:CP_Elec_4x5.8, symbol Device:C_Polarized_US
- added C31: 100NF, Capacitor_SMD:C_0603_1608Metric, symbol Seed3-Pedal-DevKit-Converted-eagle-import:Electrosmith-Passives_C-EUC0402
- added FB1: FERRITE_BEAD_0603, Resistor_SMD:R_0603_1608Metric, symbol Seed3-Pedal-DevKit-Converted-eagle-import:FERRITE_BEAD_0603
- added J8: Barrel_Jack_Switch, Connector_BarrelJack:BarrelJack_Wuerth_6941xx301002, symbol Connector:Barrel_Jack_Switch
- C13, C14, C21, C23, C24, C27, C43: footprint PANASONIC_D -> Capacitor_SMD:CP_Elec_6.3x7.7; symbol Seed3-Pedal-DevKit-Converted-eagle-import:C-EU-POL_D -> Device:C_Polarized_US
- C15, C26: footprint C0805 -> Capacitor_SMD:C_0805_2012Metric
- C16, C20, C22: footprint C0402 -> Capacitor_SMD:C_0603_1608Metric
- D5, D6: footprint SOD-323F_29887508 -> Diode_SMD:D_SOD-323; symbol Seed3-Pedal-DevKit-Converted-eagle-import:Electrosmith-Semiconductors_DIODE_SOD-323F -> Diode:1N4148WS
- FB10, FB2, FB3, FB4, FB5, FB7, FB8, FB9: footprint WUERTH-ELEKTRONIK_0603 -> Resistor_SMD:R_0603_1608Metric
- R48, R55, R57: footprint R0603 -> Resistor_SMD:R_0603_1608Metric
- U8: footprint SOT223 -> Package_TO_SOT_SMD:SOT-223-3_TabPin2
Connections:
- net +5V: now also C43.1, C18.1, FB1.2; no longer C43.+ (POS)
- net +9V: now also C13.1; no longer C13.+ (POS)
- net +9V_A: now also C23.1, C24.1; no longer C23.+ (POS), C24.+ (POS)
- net +9V_PRE: now also C21.1, D5.2 (A), D6.2 (A); no longer C21.+ (POS), D5.A, D6.A
- net GND: now also C13.2, C14.2, C21.2, C23.2, C24.2, C27.2, C43.2, C18.2, C19.2, C31.2; no longer C13.- (NEG), C14.- (NEG), C21.- (NEG), C23.- (NEG), C24.- (NEG), C27.- (NEG), C43.- (NEG)
- net at R57.1: now also D6.1 (K); no longer D6.C
- net at FB9.1: now also D5.1 (K); no longer D5.C
- net at C16.1, C26.1, FB2.2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: now also C27.1; no longer C27.+ (POS)
- net at R48.2, R55.1: now also C14.1; no longer C14.+ (POS)
- net at C20.1, FB10.1: now also J8.2
- net at C20.2, FB3.1: now also J8.1
- new net +5V_A: C19.1, C31.1, FB1.1
Other:
- note removed: "Ik = (Vin - VRef) / R 1.25mA = (5V - 2.5V) / 2k"
- moved on the sheet: FB9, R48, R55
