File: pcb/Seed3-Pedal-DevKit-Converted.kicad_pcb (KiCad board)
At the start: 2 copper layers, 197 x 100 mm, 136 parts, among them J10 DIN_MIDI_5P, J11 DIN_MIDI_5P, J2 JACK_TRS_SWITCHING, J3 JACK_TRS_SWITCHING, J4 JACK_TRS_SWITCHING, J5 JACK_TRS_SWITCHING, J6 JACK_TRS_SWITCHING, J7 GUITAR_DC_JACK, J8 USB-C31-S-RA-CS2-SMT-BK-T/R, Q1 3904, Q5 3904, SW1 TOGGLE_ON_OFF_ON_PIP2, SW2 TOGGLE_ON-ON_PIP3, SW3 SMT Mini Button, U14 USBLC6-2SC6, U2 OPTOISOLATOR_H11L1M, U3 MCP6024, U4 LM4040DBZ-2.5, U5 V23_RELAY_EE2, U6 V23_RELAY_EE2, U7 MICRO_SD_CARD, U8 LD1117-5V

Commit message: everything's on the board.
Parts:
- removed C40: 100UF DNI, PANASONIC_D
- removed C58: 10UF, PANASONIC_B
- removed D2: NSR1020MW2T3G, SOD-323F
- removed FB6: FERRITE_BEAD_0603, WUERTH-ELEKTRONIK_0603
- removed FD4, FD5, FD6: FIDUCIAL, FIDUCIAL_1MM
- removed J7: GUITAR_DC_JACK, WQP-DC0500
- removed U2: OPTOISOLATOR_H11L1M, DIL06_GULLWING
- added C17: 100NF, Capacitor_SMD:C_0603_1608Metric, F.Cu at (118.8, 127.3)
- added C25: 100NF, Capacitor_SMD:C_0603_1608Metric, F.Cu at (132.3, 106.0)
- added C28: 1NF, Capacitor_SMD:C_0603_1608Metric, F.Cu at (145.0, 106.2)
- added C29: 10uF, Capacitor_SMD:CP_Elec_4x5.8, F.Cu at (145.8, 98.5)
- added C30: 1NF, Capacitor_SMD:C_0603_1608Metric, F.Cu at (137.6, 108.3)
- added C31: 100NF, Capacitor_SMD:C_0603_1608Metric, F.Cu at (213.1, 83.8)
- added C32: 270PF, Capacitor_SMD:C_0603_1608Metric, F.Cu at (131.5, 103.5)
- added C35: 10uF, Capacitor_SMD:CP_Elec_4x5.8, F.Cu at (131.4, 109.2)
- added C37: 33NF, Capacitor_SMD:C_0603_1608Metric, F.Cu at (132.3, 101.2)
- added C38: 100PF, Capacitor_SMD:C_0603_1608Metric, F.Cu at (116.4, 120.0)
- added C42: 10uF, Capacitor_SMD:CP_Elec_4x5.8, F.Cu at (123.2, 123.3)
- added C48: 10uF, Capacitor_SMD:CP_Elec_4x5.8, F.Cu at (108.4, 123.7)
- added FB1: FERRITE_BEAD_0603, Resistor_SMD:R_0603_1608Metric, F.Cu at (209.9, 83.8)
- added FSW_2: M12 SPST Footswitch Assembly, parts-for-kicad:S02P, F.Cu at (188.0, 145.0)
- added J1: DIN_MIDI_5P, parts-for-kicad:57PC5F, F.Cu at (235.0, 100.0)
- added R28: 10R, Resistor_SMD:R_0603_1608Metric, F.Cu at (227.8, 95.0)
- added R29: 10R, Resistor_SMD:R_0603_1608Metric, F.Cu at (227.9, 105.1)
- added R58: 3K3, Resistor_SMD:R_0603_1608Metric, F.Cu at (139.3, 108.3)
- added R69: 10K, Resistor_SMD:R_0603_1608Metric, F.Cu at (129.9, 103.5)
- added R7: 1M, Resistor_SMD:R_0603_1608Metric, F.Cu at (145.8, 103.8)
- added R70: 10K, Resistor_SMD:R_0603_1608Metric, F.Cu at (133.1, 103.5)
- added R71: 4K7, Resistor_SMD:R_0603_1608Metric, F.Cu at (135.9, 108.3)
- added R72: 100R, Resistor_SMD:R_0603_1608Metric, F.Cu at (135.5, 100.0)
- added R74: 15K, Resistor_SMD:R_0603_1608Metric, F.Cu at (116.4, 118.5)
- added R75: 24K, Resistor_SMD:R_0603_1608Metric, F.Cu at (116.4, 121.7)
- added R76: 100R, Resistor_SMD:R_0603_1608Metric, F.Cu at (118.7, 122.5)
- added R77: 10K, Resistor_SMD:R_0603_1608Metric, F.Cu at (122.4, 119.8)
- added R8: 100R, Resistor_SMD:R_0603_1608Metric, F.Cu at (144.2, 103.8)
- added SW4: PTH Mini Button, parts-for-kicad:TL1105SPF250Q, F.Cu at (152.0, 145.0)
- added SW6: TOGGLE_ON-ON_PIP3, parts-for-kicad:TOGGLE_SILK_PIP3, F.Cu at (116.0, 145.0)
- added U1: MCP6002-xSN, Package_SO:SOIC-8_5.275x5.275mm_P1.27mm, F.Cu at (88.5, 101.8)
- added U10: OPA1652, Package_SO:SOIC-8_5.275x5.275mm_P1.27mm, F.Cu at (115.0, 127.2)
- added U11: H11L1, Package_DIP:DIP-6_W7.62mm, F.Cu at (230.2, 137.5)
- added U9: OPA1652, Package_SO:SOIC-8_5.275x5.275mm_P1.27mm, F.Cu at (138.6, 103.8)
- added VR4: P-10K-B-R-PIP, parts-for-kicad:9MM_SNAP-IN_POT_SILK_PIP, F.Cu at (170.0, 125.0)
- added VR5: P-10K-B-R-PIP, parts-for-kicad:9MM_SNAP-IN_POT_SILK_PIP, F.Cu at (188.0, 125.0)
- added VR6: P-10K-B-R-PIP, parts-for-kicad:9MM_SNAP-IN_POT_SILK_PIP, F.Cu at (206.0, 125.0)
- C1, C16, C20, C22, C33, C34, C47: footprint C0402 -> Capacitor_SMD:C_0603_1608Metric
- C10: value 470pF -> 10uF; footprint C0603_29888544 -> Capacitor_SMD:CP_Elec_4x5.8
- C11: value 470pF -> 270PF; footprint C0603_29888544 -> Capacitor_SMD:C_0603_1608Metric
- C12: value 10UF -> 33NF; footprint C0805 -> Capacitor_SMD:C_0603_1608Metric
- C13, C14, C21, C23, C24, C27, C36, C39, C41, C43: footprint PANASONIC_D -> Capacitor_SMD:CP_Elec_6.3x7.7
- C15, C26: footprint C0805 -> Capacitor_SMD:C_0805_2012Metric
- C18: footprint PANASONIC_B -> Capacitor_SMD:CP_Elec_4x5.8
- C19: value 100NF -> 10UF; footprint C0402_29888544 -> Capacitor_SMD:CP_Elec_4x5.8
- C2, C4: footprint C0402_29888544 -> Capacitor_SMD:C_0603_1608Metric
- C3: value 10UF -> 10uF; footprint C0805 -> Capacitor_SMD:CP_Elec_4x5.8
- C46, C55: footprint C0603 -> Capacitor_SMD:C_0603_1608Metric
- C5: value 100NF -> 100PF; footprint C0402_29888544 -> Capacitor_SMD:C_0603_1608Metric
- C6: value 330PF -> 10uF; footprint C0603 -> Capacitor_SMD:CP_Elec_4x5.8
- C7: value 100NF -> 10uF; footprint C0402_29888544 -> Capacitor_SMD:CP_Elec_4x5.8
- C8: value 10UF -> 1NF; footprint PANASONIC_B -> Capacitor_SMD:C_0603_1608Metric
- C9: value 1500PF -> 1NF; footprint C0603_29888544 -> Capacitor_SMD:C_0603_1608Metric
- D3, D4: footprint SOD-323F -> Diode_SMD:D_SOD-323
- D5, D6: footprint SOD-323F_29887508 -> Diode_SMD:D_SOD-323
- FB10, FB2, FB3, FB4, FB5, FB7, FB8, FB9: footprint WUERTH-ELEKTRONIK_0603 -> Resistor_SMD:R_0603_1608Metric
- FD1, FD2, FD3: footprint FIDUCIAL_1MM -> Fiducial:Fiducial_1mm_Mask2mm
- FSW_1: footprint S02P -> parts-for-kicad:S02P
- H1, H2, H3, H4: footprint 35-PAD -> MountingHole:MountingHole_3.5mm_Pad
- J10, J11: footprint 57PC5F -> parts-for-kicad:57PC5F
- J2, J3, J4, J5, J6: footprint TRS_JACK_WQP-PJ609B -> parts-for-kicad:TRS_JACK_WQP-PJ609B
- J8: value USB-C31-S-RA-CS2-SMT-BK-T/R -> Barrel_Jack_Switch; footprint ADAM_USB-C31-S-RA-CS2-SMT-BK-T_R -> Connector_BarrelJack:BarrelJack_Wuerth_6941xx301002
- L2: footprint SDR0805 -> parts-for-kicad:SDR0805
- LED1: value LED_RED_0603 -> LED; footprint DIODE_0603 -> LED_THT:LED_D5.0mm
- LED2: value RGB LED SMT PLCC4 -> LED_RKBG; footprint P-LCC-4-3 -> LED_THT:LED_D5.0mm-4_RGB
- LOGO1: footprint OSHW-LOGO-L_TEXT -> parts-for-kicad:OSHW-LOGO-L_TEXT
- Q1, Q5: footprint SOT23-BEC -> Package_TO_SOT_SMD:SOT-23
- R1, R17, R18, R2, R25, R3, R4, R40, R43, R44, R46, R48, R5, R50, R51, R52, R53, R54, R55, R57, R59, R60, R61, R64, R65, R68: footprint R0603 -> Resistor_SMD:R_0603_1608Metric
- R10, R23, R24, R9: footprint R0603_29888544 -> Resistor_SMD:R_0603_1608Metric
- R11: value 2M -> 15K; footprint R0603 -> Resistor_SMD:R_0603_1608Metric
- R12: value 10K -> 24K; footprint R0603 -> Resistor_SMD:R_0603_1608Metric
- R13: value 10K -> 100R; footprint R0603 -> Resistor_SMD:R_0603_1608Metric
- R14: value 100R -> 10K; footprint R0603 -> Resistor_SMD:R_0603_1608Metric
- R15: value 10K -> 1M; footprint R0603 -> Resistor_SMD:R_0603_1608Metric
- R16: value 2M -> 100R; footprint R0603 -> Resistor_SMD:R_0603_1608Metric
- R19: value 1M DNI -> 10K; footprint R0603 -> Resistor_SMD:R_0603_1608Metric
- R20: value 2M -> 3K3; footprint R0603 -> Resistor_SMD:R_0603_1608Metric
- R21: value 10K -> 4K7; footprint R0603 -> Resistor_SMD:R_0603_1608Metric
- R22: value 2M -> 10K; footprint R0603 -> Resistor_SMD:R_0603_1608Metric
- R26: value 20K -> 10K; footprint R0603 -> Resistor_SMD:R_0603_1608Metric
- R27: value 15K -> 100R; footprint R0603 -> Resistor_SMD:R_0603_1608Metric
- R56: value 0R -> 10K; footprint R0603 -> Resistor_SMD:R_0603_1608Metric
- R62, R63: footprint R0805 -> Resistor_SMD:R_0603_1608Metric
- SW1, SW2: footprint TOGGLE_SILK_PIP3 -> parts-for-kicad:TOGGLE_SILK_PIP3
- SW3: value SMT Mini Button -> PTH Mini Button; footprint TL3301SPF160QJ -> parts-for-kicad:TL1105SPF250Q
- U14: footprint SOT-23-6L -> Package_TO_SOT_SMD:SOT-23-6
- U3: value MCP6024 -> OPA1652; footprint TSSOP-14_29886060 -> Package_SO:SOIC-8_5.275x5.275mm_P1.27mm
- U4: value LM4040DBZ-2.5 -> GT-USB-7010ASV; footprint Package_TO_SOT_SMD:SOT-23 -> GT-USB-7010ASV-easyeda-usbc:USB-C-SMD_G-SWITCH_GT-USB-7010ASV
- U5, U6: value V23_RELAY_EE2 -> G6K-2F-Y-TR DC3; footprint EE2-3SNU-L -> PCB_PCB_relays_2025-01-13:RELAY-SMD_G6K-2F-Y
- U7: footprint MEM2061-01-188-00-A_GCT -> parts-for-kicad:MEM2061-01-188-00-A_GCT
- U8: footprint SOT223 -> Package_TO_SOT_SMD:SOT-223-3_TabPin2
- VR1, VR2, VR3: footprint 9MM_SNAP-IN_POT_SILK_PIP -> parts-for-kicad:9MM_SNAP-IN_POT_SILK_PIP
- moved LED1 126.1 mm to (206.0, 146.0), turned to 90 degrees
- moved R43 124.7 mm to (200.6, 141.8)
- moved C19 116.9 mm to (212.6, 88.2), turned to -90 degrees
- moved C18 111.9 mm to (207.4, 88.2), turned to -90 degrees
- moved C6 63.8 mm to (123.3, 131.2), turned to 180 degrees
- moved C4 59.5 mm to (107.4, 105.5), turned to 180 degrees
- moved U4 58.4 mm to (195.0, 60.0), turned to 180 degrees
- moved SW3 56.0 mm to (134.0, 145.0)
- moved R11 54.0 mm to (114.8, 136.2), turned to 180 degrees
- moved C27 53.0 mm to (198.6, 80.0), turned to 90 degrees
- moved C5 52.6 mm to (114.8, 134.6), turned to 0 degrees
- moved FSW_1 52.1 mm to (170.0, 145.0)
- moved D6 49.7 mm to (189.2, 77.2), turned to 180 degrees
- moved C8 49.1 mm to (120.0, 105.9), turned to 0 degrees
- moved R14 48.8 mm to (122.4, 134.8), turned to 180 degrees
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Connections:
- A1 pad 1: unconnected-(A1-USB_ID-Pad1) -> TAC_SW
- A1 pad 10: unconnected-(A1-SPI1_POCI-Pad10) -> TOG_1
- A1 pad 11: unconnected-(A1-SPI1_PICO-Pad11) -> GPIO_FSW_1
- A1 pad 12: unconnected-(A1-I2C1_SCL-Pad12) -> /ES_Daisy_Seed2_DFM_EVAL_PEDAL_Rev5_1/GPIO_RELAY_L
- A1 pad 13: unconnected-(A1-I2C1_SDA-Pad13) -> /ES_Daisy_Seed2_DFM_EVAL_PEDAL_Rev5_1/GPIO_RELAY_R
- A1 pad 14: unconnected-(A1-USART1_TX-Pad14) -> MIDI_TX
- A1 pad 15: unconnected-(A1-USART1_RX-Pad15) -> MIDI_RX
- A1 pad 16: unconnected-(A1-AUDIO_IN_1-Pad16) -> CODEC_IN_L
- A1 pad 17: unconnected-(A1-AUDIO_IN_2-Pad17) -> CODEC_IN_R
- A1 pad 18: unconnected-(A1-AUDIO_OUT_1-Pad18) -> CODEC_OUT_L
- A1 pad 19: unconnected-(A1-AUDIO_OUT_2-Pad19) -> CODEC_OUT_R
- A1 pad 2: unconnected-(A1-SD_DATA_3-Pad2) -> SDMMC_D3
- A1 pad 22: unconnected-(A1-ADC_0-Pad22) -> POT_1
- A1 pad 23: unconnected-(A1-ADC_1-Pad23) -> POT_2
- A1 pad 24: unconnected-(A1-ADC_2-Pad24) -> POT_3
- A1 pad 25: unconnected-(A1-ADC_3-Pad25) -> POT_4
- A1 pad 26: unconnected-(A1-ADC_4-Pad26) -> POT_5
- A1 pad 27: unconnected-(A1-ADC_5-Pad27) -> POT_6
- A1 pad 28: unconnected-(A1-ADC_6-Pad28) -> ADC_EXPRESSION
- A1 pad 29: unconnected-(A1-DAC_OUT2-Pad29) -> TOG_3
- A1 pad 3: unconnected-(A1-SD_DATA_2-Pad3) -> SDMMC_D2
- A1 pad 30: unconnected-(A1-DAC_OUT1-Pad30) -> GPIO_FSW_2
- A1 pad 31: unconnected-(A1-SAI2_MCLK-Pad31) -> LED_MONO_1
- A1 pad 32: unconnected-(A1-SAI2_SD_B-Pad32) -> LED_R
- A1 pad 33: unconnected-(A1-SAI2_SD_A-Pad33) -> LED_G
- A1 pad 34: unconnected-(A1-SAI2_FS-Pad34) -> LED_B
- A1 pad 35: unconnected-(A1-SAI2_SCK-Pad35) -> TAC_SW2
- A1 pad 36: unconnected-(A1-USB_D_--Pad36) -> /ES_Daisy_Seed2_DFM_EVAL_PEDAL_Rev5_1/USB_OTG_HS_N
- A1 pad 37: unconnected-(A1-USB_D_+-Pad37) -> /ES_Daisy_Seed2_DFM_EVAL_PEDAL_Rev5_1/USB_OTG_HS_P
- A1 pad 4: unconnected-(A1-SD_DATA_1-Pad4) -> SDMMC_D1
- A1 pad 5: unconnected-(A1-SD_DATA_0-Pad5) -> SDMMC_D0
- A1 pad 6: unconnected-(A1-SD_CMD-Pad6) -> SDMMC_CMD
- A1 pad 7: unconnected-(A1-SD_CLK-Pad7) -> SDMMC_CK
- A1 pad 8: unconnected-(A1-SPI1_CS-Pad8) -> TOG_2_B
- A1 pad 9: unconnected-(A1-SPI1_SCK-Pad9) -> TOG_2_A
- C10 pad 1: Net-(U3A-OUT) -> Net-(C10-Pad1)
- C10 pad 2: Net-(U3A--IN) -> Net-(C10-Pad2)
- C11 pad 1: Net-(U3A-+IN) -> Net-(U3B--)
- C11 pad 2: GND -> Net-(C11-Pad2)
- C12 pad 1: Net-(U3A-OUT) -> GND
- C12 pad 2: Net-(C12-Pad2) -> CODEC_IN_R
- C16 pad 1: Net-(C27-POS) -> Net-(U8-IN)
- C19 pad 1: /ES_Daisy_Seed2_DFM_EVAL_PEDAL_Rev5_3/CODEC_VCC -> +5V_A
- C2 pad 1: /ES_Daisy_Seed2_DFM_EVAL_PEDAL_Rev5_3/CODEC_VCC -> +5V_A
- C20 pad 1: Net-(J7-PIN) -> Net-(C20-Pad1)
- C26 pad 1: Net-(C27-POS) -> Net-(U8-IN)
- C3 pad 1: Net-(U3B-OUT) -> Net-(C3-Pad1)
- C3 pad 2: Net-(C3-Pad2) -> CODEC_OUT_R
- C33 pad 1: /ES_Daisy_Seed2_DFM_EVAL_PEDAL_Rev5_3/+2V5_PRE -> Net-(U1A-+)
- C4 pad 1: /ES_Daisy_Seed2_DFM_EVAL_PEDAL_Rev5_3/CODEC_VCC -> +9V_A
- C5 pad 1: Net-(C5-Pad1) -> Net-(U10B--)
- C5 pad 2: Net-(Q3-G) -> Net-(C5-Pad2)
- C55 pad 1: /ES_Daisy_Seed2_DFM_EVAL_PEDAL_Rev5_3/+2V5_PRE -> Net-(U1A-+)
- C6 pad 1: Net-(U3D-OUT) -> AUDIO_DSP_RIGHT
- C6 pad 2: Net-(U3D--IN) -> Net-(C6-Pad2)
- C7 pad 1: GND -> Net-(C7-Pad1)
- C7 pad 2: /ES_Daisy_Seed2_DFM_EVAL_PEDAL_Rev5_3/AREF_+2V5 -> AUDIO_BUFF_RIGHT
- C9 pad 1: Net-(C9-Pad1) -> Net-(C10-Pad2)
- C9 pad 2: Net-(C9-Pad2) -> GND
- FB10 pad 1: Net-(J7-PIN) -> Net-(C20-Pad1)
- FB2 pad 2: Net-(C27-POS) -> Net-(U8-IN)
- FB9 pad 1: Net-(D5-PadC) -> Net-(D5-K)
- L2 pad P$1: Net-(C41-POS) -> Net-(C41-Pad1)
- LED2 pad 2: +3V3 -> GND
- R1 pad 1: Net-(J8-CC2) -> Net-(U4-CC1)
- R10 pad 1: Net-(Q1-PadB) -> Net-(Q1-B)
- R11 pad 1: +5V -> Net-(U10B--)
- R11 pad 2: Net-(Q2-G) -> Net-(C3-Pad1)
- R12 pad 1: Net-(C66-Pad1) -> Net-(C5-Pad2)
- R12 pad 2: CODEC_OUT_L_N -> Net-(U10B--)
- R13 pad 1: Net-(C31-POS) -> Net-(C6-Pad2)
- R13 pad 2: GND -> Net-(C5-Pad2)
- R14 pad 1: AUDIO_DSP_LEFT -> AUDIO_DSP_RIGHT
- R14 pad 2: Net-(C3-Pad2) -> GND
- R15 pad 1: GND -> Net-(C7-Pad1)
- R15 pad 2: Net-(C3-Pad2) -> +5V_A
- R16 pad 1: Net-(Q2-G) -> Net-(U3A-+)
- R16 pad 2: GND -> Net-(C7-Pad1)
- R19 pad 1: /ES_Daisy_Seed2_DFM_EVAL_PEDAL_Rev5_3/+2V5_PRE -> Net-(U1A-+)
- R2 pad 2: Net-(J8-CC1) -> Net-(U4-CC2)
- R20 pad 1: +5V -> Net-(C10-Pad2)
- R20 pad 2: Net-(Q3-G) -> Net-(U3A--)
- R21 pad 1: Net-(C8-POS) -> Net-(C10-Pad2)
- R22 pad 1: Net-(Q3-G) -> Net-(U3B--)
- R22 pad 2: GND -> Net-(C10-Pad1)
- R23 pad 2: Net-(Q5-PadB) -> Net-(Q5-B)
- R24 pad 1: Net-(Q5-PadB) -> Net-(Q5-B)
- R26 pad 1: Net-(U3D--IN) -> Net-(C11-Pad2)
- R26 pad 2: Net-(C8-NEG) -> Net-(U3B--)
- R27 pad 1: Net-(U3D-OUT) -> CODEC_IN_R
- R27 pad 2: Net-(U3D--IN) -> Net-(C11-Pad2)
- R3 pad 1: /ES_Daisy_Seed2_DFM_EVAL_PEDAL_Rev5_1/MIDI_RX -> MIDI_RX
- R43 pad 2: Net-(LED1-C) -> Net-(LED1-A)
- R46 pad 2: +5V -> +5V_A
- R48 pad 2: Net-(C14-POS) -> Net-(C14-Pad1)
- R5 pad 1: /ES_Daisy_Seed2_DFM_EVAL_PEDAL_Rev5_3/AREF_+2V5 -> /ES_Daisy_Seed2_DFM_EVAL_PEDAL_Rev5_3/AREF_AUDIO_IN_BIAS
- R55 pad 1: Net-(C14-POS) -> Net-(C14-Pad1)
- R56 pad 1: AREF_2v5_PRE -> +3V3_A
- R56 pad 2: /ES_Daisy_Seed2_DFM_EVAL_PEDAL_Rev5_3/+2V5_PRE -> Net-(U1A-+)
- R57 pad 1: Net-(D6-PadC) -> Net-(D6-K)
- R62 pad 2: Net-(C41-POS) -> Net-(C41-Pad1)
- R63 pad 2: Net-(C41-POS) -> Net-(C41-Pad1)
- R9 pad 2: Net-(Q1-PadB) -> Net-(Q1-B)
- SW3 pad 1: TAC_SW -> TAC_SW1
- SW3 pad 2: TAC_SW -> TAC_SW1
- U3 pad 1: Net-(U3A-OUT) -> Net-(U3A--)
- U3 pad 2: Net-(U3A--IN) -> Net-(U3A--)
- U3 pad 3: Net-(U3A-+IN) -> Net-(U3A-+)
- U3 pad 4: /ES_Daisy_Seed2_DFM_EVAL_PEDAL_Rev5_3/CODEC_VCC -> GND
- U3 pad 5: Net-(U3B-+IN) -> /ES_Daisy_Seed2_DFM_EVAL_PEDAL_Rev5_3/AREF_AUDIO_IN_BIAS
- U3 pad 6: Net-(U3B--IN) -> Net-(U3B--)
- U3 pad 7: Net-(U3B-OUT) -> Net-(C11-Pad2)
- U3 pad 8: Net-(U3C-OUT) -> +9V_A
- U4 pad 1: AREF_2v5_PRE -> GND
- U4 pad 3: unconnected-(U4-NC-Pad3) -> GND
- U5 pad 1: Net-(D3-PadA) -> +3V3
- U5 pad 3: AUDIO_OUT_LEFT -> AUDIO_DSP_LEFT
- U5 pad 4: AUDIO_IN_LEFT -> AUDIO_OUT_LEFT
- U5 pad 8: AUDIO_OUT_LEFT -> Net-(D3-A)
- U6 pad 1: Net-(D4-PadA) -> +3V3
- U6 pad 3: AUDIO_OUT_RIGHT -> AUDIO_DSP_RIGHT
- U6 pad 4: AUDIO_IN_RIGHT -> AUDIO_OUT_RIGHT
- U6 pad 8: AUDIO_OUT_RIGHT -> Net-(D4-A)
- U8 pad 3: Net-(C27-POS) -> Net-(U8-IN)
Routing:
- net +9V_A: track 91.5 -> 0.00 mm, vias 4 -> 0
- net AUDIO_OUT_RIGHT: track 79.5 -> 0.00 mm, vias 2 -> 0
- net AUDIO_OUT_LEFT: track 74.7 -> 0.00 mm, vias 2 -> 0
- net +9V_PRE: track 71.7 -> 0.00 mm, vias 2 -> 0
- net /ES_Daisy_Seed2_DFM_EVAL_PEDAL_Rev5_3/AREF_+2V5: track 68.7 -> 0.00 mm, vias 2 -> 0
- net /ES_Daisy_Seed2_DFM_EVAL_PEDAL_Rev5_3/CODEC_VCC: track 66.1 -> 0.00 mm, vias 4 -> 0
- net AUDIO_DSP_RIGHT: track 58.8 -> 0.00 mm, vias 4 -> 0
- net Net-(C31-POS): track 52.0 -> 0.00 mm, vias 2 -> 0
- net Net-(C8-POS): track 45.5 -> 0.00 mm, vias 4 -> 0
- net SDMMC_CMD: track 0.00 -> 29.8 mm
- net Net-(J7-PIN): track 22.4 -> 0.00 mm
- net /ES_Daisy_Seed2_DFM_EVAL_PEDAL_Rev5_3/+2V5_PRE: track 21.3 -> 0.00 mm
- net SDMMC_CK: track 0.00 -> 20.2 mm
- net AUDIO_IN_LEFT: track 16.9 -> 0.00 mm, vias 1 -> 0
- net /ES_Daisy_Seed2_DFM_EVAL_PEDAL_Rev5_1/+9V_FILT: track 16.6 -> 0.00 mm
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Other:
- board text added: "(C) Electrosmith 2025"
- board text added: "MIDI THRU"
- board text added: "Seed3 Pedal Dev Kit"
- board text removed: "(C) Electrosmith 2023"
- board text removed: "Daisy Seed2 DFM EVAL PEDAL Rev5"
