File: pcb/Seed3-Pedal-DevKit-Converted.kicad_pcb (KiCad board)
At the start: 2 copper layers, 197 x 100 mm, 164 parts, among them J1 DIN_MIDI_5P, J10 DIN_MIDI_5P, J11 DIN_MIDI_5P, J2 JACK_TRS_SWITCHING, J3 JACK_TRS_SWITCHING, J4 JACK_TRS_SWITCHING, J5 JACK_TRS_SWITCHING, J6 JACK_TRS_SWITCHING, J8 Barrel_Jack_Switch, Q1 3904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

Commit message: first round of gerbs.
Parts:
- added REF**: WEEE-Logo_4.2x6mm_SilkScreen, Symbol:WEEE-Logo_4.2x6mm_SilkScreen, B.Cu at (213.7, 140.5)
- added REF**: RoHS-Logo_6mm_SilkScreen, Symbol:RoHS-Logo_6mm_SilkScreen, B.Cu at (221.8, 148.0)
- LED2: footprint LED_THT:LED_D5.0mm-4_RGB -> LED_THT:LED_D5.0mm-4_RGB_Wide_Pins
- SW3, SW4: value PTH Mini Button -> SMT Mini Button; footprint parts-for-kicad:TL1105SPF250Q -> parts-for-kicad:TL3301SPF160QJ
- moved LED2 1.09 mm to (80.0, 132.0)
- turned SW3 to 180 degrees
- turned SW4 to 180 degrees
Routing:
- net SDMMC_CMD: track 29.8 -> 20.5 mm, vias 0 -> 1
- net SDMMC_CK: track 18.5 -> 26.5 mm
- net SDMMC_D1: track 11.9 -> 17.4 mm
- net SDMMC_D0: track 14.2 -> 16.5 mm
- net Net-(C41-Pad1): track 16.0 -> 14.8 mm
- net TAC_SW2: track 113.7 -> 112.6 mm
- net TAC_SW1: track 102.7 -> 101.8 mm
- net Net-(U9A-+): track 4.28 -> 3.60 mm
- net Net-(LED2-GA): track 11.6 -> 12.3 mm
- net AUDIO_OUT_RIGHT: track 65.5 -> 64.9 mm
- net +5V: track 24.2 -> 23.6 mm
- net TOG_2_A: track 26.0 -> 25.4 mm
- net Net-(C48-Pad1): track 7.85 -> 7.30 mm
- net +9V_A: track 135.4 -> 134.9 mm
Other:
- board text added: "0"
- board text added: "0 mm"
- board text added: "0.0000 mm / 0.1524 mm"
- board text added: "0.01 mm"
- board text added: "0.02"
- board text added: "0.035 mm"
- board text added: "0.3000 mm"
- board text added: "1"
- board text added: "1.51 mm"
- board text added: "1.6000 mm"
- board text added: "197.0000 mm x 100.0000 mm"
- board text added: "2"
- board text added: "3.3"
- board text added: "4.5"
- board text added: "B.Cu"
- board text added: "B.Mask"
- board text added: "B.Paste"
- board text added: "B.Silkscreen"
- board text added: "BOARD CHARACTERISTICS"
- board text added: "Board Thickness:"
- board text added: "Board overall dimensions:"
- board text added: "Bottom Silk Screen"
- board text added: "Bottom Solder Mask"
- board text added: "Bottom Solder Paste"
- board text added: "Castellated pads:"
- board text added: "Color"
- board text added: "Copper Finish:"
- board text added: "Copper Layer Count:"
- board text added: "Dielectric"
- board text added: "Edge card connectors:"
- board text added: "Epsilon R"
- board text added: "F.Cu"
- board text added: "F.Mask"
- board text added: "F.Paste"
- board text added: "F.Silkscreen"
- board text added: "FR4"
- board text added: "Impedance Control:"
- board text added: "Layer Name"
- board text added: "Loss Tangent"
- board text added: "Material"
- board text added: "Min hole diameter:"
- board text added: "Min track/spacing:"
- board text added: "No"
- board text added: "None"
- board text added: "Not specified"
- board text added: "Plated Board Edge:"
- board text added: "Thickness (mm)"
- board text added: "Top Silk Screen"
- board text added: "Top Solder Mask"
- board text added: "Top Solder Paste"
- board text added: "Type"
- board text added: "copper"
- board text added: "core"
