File: pcb/ES_Daisy_Seed2_DFM_EVAL_PEDAL_Rev5_1.kicad_sch (KiCad schematic)
At the start: 36 parts, among them J8 USB-C31-S-RA-CS2-SMT-BK-T/R, Q1 3904, Q5 3904, U14 USBLC6-2SC6, U2 OPTOISOLATOR_H11L1M, U5 V23_RELAY_EE2, U6 V23_RELAY_EE2

Commit message: everything's on the board.
Parts:
- removed D2: NSR1020MW2T3G, SOD-323F, symbol Seed3-Pedal-DevKit-Converted-eagle-import:Electrosmith-Semiconductors_DIODE_SOD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
- removed FD4, FD5, FD6: FIDUCIAL, FIDUCIAL_1MM, symbol Seed3-Pedal-DevKit-Converted-eagle-import:FIDUCIAL
- removed J8: USB-C31-S-RA-CS2-SMT-BK-T/R, ADAM_USB-C31-S-RA-CS2-SMT-BK-T_R, symbol Seed3-Pedal-DevKit-Converted-eagle-import:USB-C31-S-RA-CS2-SMT-BK-T/R
- removed U2: OPTOISOLATOR_H11L1M, DIL06_GULLWING, symbol Seed3-Pedal-DevKit-Converted-eagle-import:OPTOISOLATOR_H11L1M
- added U11: H11L1, Package_DIP:DIP-6_W7.62mm, symbol Isolator:H11L1
- added U4: GT-USB-7010ASV, GT-USB-7010ASV-easyeda-usbc:USB-C-SMD_G-SWITCH_GT-USB-7010ASV, symbol SCH_GT-USB-7010ASV:GT-USB-7010ASV
- C1: footprint C0402 -> Capacitor_SMD:C_0603_1608Metric
- C36, C41: footprint PANASONIC_D -> Capacitor_SMD:CP_Elec_6.3x7.7; symbol Seed3-Pedal-DevKit-Converted-eagle-import:C-EU-POL_D -> Device:C_Polarized_US
- D3, D4: footprint SOD-323F -> Diode_SMD:D_SOD-323; symbol Seed3-Pedal-DevKit-Converted-eagle-import:Electrosmith-Semiconductors_DIODE_SOD-323F -> Diode:1N4148WS
- FD1, FD2, FD3: footprint FIDUCIAL_1MM -> Fiducial:Fiducial_1mm_Mask2mm
- H1, H2, H3, H4: footprint 35-PAD -> MountingHole:MountingHole_3.5mm_Pad
- L2: footprint SDR0805 -> parts-for-kicad:SDR0805
- LOGO1: footprint OSHW-LOGO-L_TEXT -> parts-for-kicad:OSHW-LOGO-L_TEXT
- Q1, Q5: footprint SOT23-BEC -> Package_TO_SOT_SMD:SOT-23; symbol Seed3-Pedal-DevKit-Converted-eagle-import:-NPN-SOT23-BEC -> Transistor_BJT:MMBT3904
- R1, R2, R3, R4: footprint R0603 -> Resistor_SMD:R_0603_1608Metric
- R10, R23, R24, R9: footprint R0603_29888544 -> Resistor_SMD:R_0603_1608Metric
- R62, R63: footprint R0805 -> Resistor_SMD:R_0603_1608Metric
- U14: footprint SOT-23-6L -> Package_TO_SOT_SMD:SOT-23-6
- U5, U6: value V23_RELAY_EE2 -> G6K-2F-Y-TR DC3; footprint EE2-3SNU-L -> PCB_PCB_relays_2025-01-13:RELAY-SMD_G6K-2F-Y; symbol Seed3-Pedal-DevKit-Converted-eagle-import:V23_RELAY_EE2 -> Relay:G6K-2
Connections:
- net +3V3: now also D3.1 (K), D4.1 (K), U5.1, U6.1, U11.6; no longer D3.C, D4.C, U5.12 (8), U6.12 (8)
- net +5V_USB: now also U4.A4B9 (VBUS), U4.B4A9 (VBUS)
- net +9V_FILT: now also C36.1; no longer C36.+ (POS)
- net ADC_EXPRESSION: now also A1.28 (ADC_6)
- net AUDIO_DSP_LEFT: now also U5.3; no longer U5.9 (7)
- net AUDIO_DSP_RIGHT: now also U6.3; no longer U6.9 (7)
- net AUDIO_IN_LEFT: now also U5.6; no longer U5.4 (2)
- net AUDIO_IN_RIGHT: now also U6.6; no longer U6.4 (2)
- net AUDIO_OUT_LEFT: now also U5.4, U5.7; no longer U5.3, U5.8 (5)
- net AUDIO_OUT_RIGHT: now also U6.4, U6.7; no longer U6.3, U6.8 (5)
- net GND: now also C36.2, C41.2, Q1.2 (E), Q5.2 (E), U11.5, U4.1 (SHELL), U4.2 (SHELL), U4.3 (SHELL), U4.4 (SHELL), U4.A1B12 (GND), U4.B1A12 (GND); no longer C36.- (NEG), C41.- (NEG), Q1.E, Q5.E
- net GPIO_FSW_1: now also A1.11 (SPI1_PICO)
- net GPIO_RELAY_L: now also A1.12 (I2C1_SCL)
- net GPIO_RELAY_R: now also A1.13 (I2C1_SDA)
- net LED_B: now also A1.34 (SAI2_FS)
- net LED_G: now also A1.33 (SAI2_SD_A)
- net LED_MONO_1: now also A1.31 (SAI2_MCLK)
- net LED_R: now also A1.32 (SAI2_SD_B)
- net MIDI_IN_5: now also U11.2
- net MIDI_RX: now also A1.15 (USART1_RX), U11.4
- net MIDI_TX: now also A1.14 (USART1_TX)
- net POT_1: now also A1.22 (ADC_0)
- net POT_2: now also A1.23 (ADC_1)
- net POT_3: now also A1.24 (ADC_2)
- net POT_4: now also A1.25 (ADC_3)
- net POT_5: now also A1.26 (ADC_4)
- net POT_6: now also A1.27 (ADC_5)
- net SDMMC_CK: now also A1.7 (SD_CLK)
- net SDMMC_CMD: now also A1.6 (SD_CMD)
- net SDMMC_D0: now also A1.5 (SD_DATA_0)
- net SDMMC_D1: now also A1.4 (SD_DATA_1)
- net SDMMC_D2: now also A1.3 (SD_DATA_2)
- net SDMMC_D3: now also A1.2 (SD_DATA_3)
- net TAC_SW: now also A1.1 (USB_ID)
- net TAC_SW2: now also A1.35 (SAI2_SCK)
- net TOG_1: now also A1.10 (SPI1_POCI)
- net TOG_2_A: now also A1.9 (SPI1_SCK)
- net TOG_2_B: now also A1.8 (SPI1_CS)
- net TOG_3: now also A1.29 (DAC_OUT2)
- net USB_IN_N: now also U4.A7 (DN1), U4.B7 (DN2)
- net USB_IN_P: now also U4.A6 (DP1), U4.B6 (DP2)
- net USB_OTG_HS_N: now also A1.36 (USB_D_-)
- net USB_OTG_HS_P: now also A1.37 (USB_D_+)
- net at R10.1, R9.2: now also Q1.1 (B); no longer Q1.B
- net at R2.2: now also U4.B5 (CC2)
- net at R1.1: now also U4.A5 (CC1)
- net at R4.2: now also U11.1
- net at R23.2, R24.1: now also Q5.1 (B); no longer Q5.B
- net at L2.P$1, R62.2, R63.2: now also C41.1; no longer C41.+ (POS)
- net CODEC_IN_L: now reaches A1.16 (AUDIO_IN_1)
- net CODEC_IN_R: now reaches A1.17 (AUDIO_IN_2)
- net CODEC_OUT_L: now reaches A1.18 (AUDIO_OUT_1)
- net CODEC_OUT_R: now reaches A1.19 (AUDIO_OUT_2)
- net GPIO_FSW_2: now reaches A1.30 (DAC_OUT1)
- new net: D3.2 (A), Q1.3 (C), U5.8
- new net: D4.2 (A), Q5.3 (C), U6.8
Other:
- moved on the sheet: C1, R1, R2, R3, R4, U14

Commit message: fully routed.
Connections:
- net LED_B: now also A1.33 (SAI2_SD_A); no longer A1.34 (SAI2_FS)
- net LED_G: now also A1.34 (SAI2_FS); no longer A1.33 (SAI2_SD_A)
- net TAC_SW renamed TAC_SW1
Changed lines of the file:
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@@
 		)
 	)
-	(global_label "TAC_SW"
+	(global_label "TAC_SW1"
 		(shape bidirectional)
 		(at 138.43 78.74 0)
@@
 		)
 		(property "Intersheetrefs" "${INTERSHEET_REFS}"
-			(at 149.2599 78.74 0)
+			(at 150.4452 78.74 0)
 			(effects
 				(font
@@
 	(global_label "LED_G"
 		(shape bidirectional)
+		(at 76.2 128.27 180)
+		(fields_autoplaced yes)
+		(effects
+			(font
+				(size 1.2446 1.2446)
+			)
+			(justify right)
+		)
+		(property "Intersheetrefs" "${INTERSHEET_REFS}"
+			(at 66.6147 128.27 0)
+			(effects
+				(font
+					(size 1.27 1.27)
+				)
+				(justify right)
+				(hide yes)
+			)
+		)
+	)
+	(global_label "AUDIO_DSP_LEFT"
+		(shape bidirectional)
+		(at 288.29 209.55 0)
+		(fields_autoplaced yes)
+		(effects
+			(font
+				(size 1.2446 1.2446)
+			)
+			(justify left)
+		)
+		(property "Intersheetrefs" "${INTERSHEET_REFS}"
+			(at 307.5359 209.55 0)
+			(effects
+				(font
+					(size 1.27 1.27)
+				)
+				(justify left)
+				(hide yes)
+			)
+		)
+	)
+	(global_label "POT_6"
+		(shape bidirectional)
+		(at 76.2 107.95 180)
+		(fields_autoplaced yes)
+		(effects
+			(font
+				(size 1.2446 1.2446)
+			)
+			(justify right)
+		)
+		(property "Intersheetrefs" "${INTERSHEET_REFS}"
+			(at 66.5554 107.95 0)
+			(effects
+				(font
+					(size 1.27 1.27)
+				)
+				(justify right)
+				(hide yes)
+			)
+		)
+	)
+	(global_label "+9V"
+		(shape bidirectional)
+		(at 43.18 46.99 180)
+		(fields_autoplaced yes)
+		(effects
+			(font
+				(size 1.2446 1.2446)
+			)
+			(justify right)
+		)
+		(property "Intersheetrefs" "${INTERSHEET_REFS}"
+			(at 35.3728 46.99 0)
+			(effects
+				(font
+					(size 1.27 1.27)
+				)
+				(justify right)
+				(hide yes)
+			)
+		)
+	)
+	(global_label "TOG_2_A"
+		(shape bidirectional)
+		(at 139.7 107.95 0)
+		(fields_autoplaced yes)
+		(effects
+			(font
+				(size 1.2446 1.2446)
+			)
+			(justify left)
+		)
+		(property "Intersheetrefs" "${INTERSHEET_REFS}"
+			(at 151.3597 107.95 0)
+			(effects
+				(font
+					(size 1.27 1.27)
+				)
+				(justify left)
+				(hide yes)
+			)
+		)
+	)
+	(global_label "SDMMC_D0"
+		(shape bidirectional)
+		(at 138.43 118.11 0)
+		(fields_autoplaced yes)
+		(effects
+			(font
+				(size 1.2446 1.2446)
+			)
+			(justify left)
+		)
+		(property "Intersheetrefs" "${INTERSHEET_REFS}"
+			(at 152.3417 118.11 0)
+			(effects
+				(font
+					(size 1.27 1.27)
+				)
+				(justify left)
+				(hide yes)
+			)
+		)
+	)
+	(global_label "AUDIO_IN_RIGHT"
+		(shape bidirectional)
+		(at 384.81 207.01 0)
+		(fields_autoplaced yes)
+		(effects
+			(font
+				(size 1.2446 1.2446)
+			)
+			(justify left)
+		)
+		(property "Intersheetrefs" "${INTERSHEET_REFS}"
+			(at 403.4634 207.01 0)
+			(effects
+				(font
+					(size 1.27 1.27)
+				)
+				(justify left)
+				(hide yes)
+			)
+		)
+	)
+	(global_label "LED_B"
+		(shape bidirectional)
 		(at 76.2 125.73 180)
 		(fields_autoplaced yes)
@@
 			(effects
 				(font
-					(size 1.27 1.27)
-				)
-				(justify right)
-				(hide yes)
-			)
-		)
-	)
-	(global_label "AUDIO_DSP_LEFT"
-		(shape bidirectional)
-		(at 288.29 209.55 0)
-		(fields_autoplaced yes)
-		(effects
-			(font
-				(size 1.2446 1.2446)
-			)
-			(justify left)
-		)
-		(property "Intersheetrefs" "${INTERSHEET_REFS}"
-			(at 307.5359 209.55 0)
-			(effects
-				(font
-					(size 1.27 1.27)
-				)
-				(justify left)
-				(hide yes)
-			)
-		)
-	)
-	(global_label "POT_6"
-		(shape bidirectional)
-		(at 76.2 107.95 180)
-		(fields_autoplaced yes)
-		(effects
-			(font
-				(size 1.2446 1.2446)
-			)
-			(justify right)
-		)
-		(property "Intersheetrefs" "${INTERSHEET_REFS}"
-			(at 66.5554 107.95 0)
-			(effects
-				(font
-					(size 1.27 1.27)
-				)
-				(justify right)
-				(hide yes)
-			)
-		)
-	)
-	(global_label "+9V"
-		(shape bidirectional)
-		(at 43.18 46.99 180)
-		(fields_autoplaced yes)
-		(effects
-			(font
-				(size 1.2446 1.2446)
-			)
-			(justify right)
-		)
-		(property "Intersheetrefs" "${INTERSHEET_REFS}"
-			(at 35.3728 46.99 0)
-			(effects
-				(font
-					(size 1.27 1.27)
-				)
-				(justify right)
-				(hide yes)
-			)
-		)
-	)
-	(global_label "TOG_2_A"
-		(shape bidirectional)
-		(at 139.7 107.95 0)
-		(fields_autoplaced yes)
-		(effects
-			(font
-				(size 1.2446 1.2446)
-			)
-			(justify left)
-		)
-		(property "Intersheetrefs" "${INTERSHEET_REFS}"
-			(at 151.3597 107.95 0)
-			(effects
-				(font
-					(size 1.27 1.27)
-				)
-				(justify left)
-				(hide yes)
-			)
-		)
-	)
-	(global_label "SDMMC_D0"
-		(shape bidirectional)
-		(at 138.43 118.11 0)
-		(fields_autoplaced yes)
-		(effects
-			(font
-				(size 1.2446 1.2446)
-			)
-			(justify left)
-		)
-		(property "Intersheetrefs" "${INTERSHEET_REFS}"
-			(at 152.3417 118.11 0)
-			(effects
-				(font
-					(size 1.27 1.27)
-				)
-				(justify left)
-				(hide yes)
-			)
-		)
-	)
-	(global_label "AUDIO_IN_RIGHT"
-		(shape bidirectional)
-		(at 384.81 207.01 0)
-		(fields_autoplaced yes)
-		(effects
-			(font
-				(size 1.2446 1.2446)
-			)
-			(justify left)
-		)
-		(property "Intersheetrefs" "${INTERSHEET_REFS}"
-			(at 403.4634 207.01 0)
-			(effects
-				(font
-					(size 1.27 1.27)
-				)
-				(justify left)
-				(hide yes)
-			)
-		)
-	)
-	(global_label "LED_B"
-		(shape bidirectional)
-		(at 76.2 128.27 180)
-		(fields_autoplaced yes)
-		(effects
-			(font
-				(size 1.2446 1.2446)
-			)
-			(justify right)
-		)
-		(property "Intersheetrefs" "${INTERSHEET_REFS}"
-			(at 66.6147 128.27 0)
-			(effects
-				(font
