File: pcb/ES_Daisy_Seed2_DFM_EVAL_PEDAL_Rev5_2.kicad_sch (KiCad schematic)
At the start: 35 parts, among them J1 DIN_MIDI_5P, J10 DIN_MIDI_5P, J11 DIN_MIDI_5P, J2 JACK_TRS_SWITCHING, J3 JACK_TRS_SWITCHING, J4 JACK_TRS_SWITCHING, J5 JACK_TRS_SWITCHING, J6 JACK_TRS_SWITCHING, SW1 TOGGLE_ON_OFF_ON_PIP2, SW2 TOGGLE_ON-ON_PIP3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

Commit message: everything's on the board.
Parts:
- removed LED1: LED_RED_0603, DIODE_0603, symbol Seed3-Pedal-DevKit-Converted-eagle-import:LED_0603
- removed LED2: RGB LED SMT PLCC4, P-LCC-4-3, symbol Seed3-Pedal-DevKit-Converted-eagle-import:LED_RGB_SMT
- added FSW_2: M12 SPST Footswitch Assembly, parts-for-kicad:S02P, symbol Seed3-Pedal-DevKit-Converted-eagle-import:SW_ASSEMBLY_CONN
- added LED1: LED, LED_THT:LED_D5.0mm, symbol Device:LED
- added LED2: LED_RKBG, LED_THT:LED_D5.0mm-4_RGB, symbol Device:LED_RKBG
- added R28, R29: 10R, Resistor_SMD:R_0603_1608Metric, symbol Seed3-Pedal-DevKit-Converted-eagle-import:Electrosmith-Passives_R-US_R0603
- added SW4: PTH Mini Button, parts-for-kicad:TL1105SPF250Q, symbol parts-for-kicad:TAC_SWITCH_PTH
- added SW6: TOGGLE_ON-ON_PIP3, parts-for-kicad:TOGGLE_SILK_PIP3, symbol Seed3-Pedal-DevKit-Converted-eagle-import:TOGGLE_ON-ON_PIP3
- added VR4, VR5, VR6: P-10K-B-R-PIP, parts-for-kicad:9MM_SNAP-IN_POT_SILK_PIP, symbol Seed3-Pedal-DevKit-Converted-eagle-import:POT_9MM_SNAP-IN__SILK_PIP
- C34, C47: footprint C0402 -> Capacitor_SMD:C_0603_1608Metric
- FSW_1: footprint S02P -> parts-for-kicad:S02P
- J1, J10, J11: footprint 57PC5F -> parts-for-kicad:57PC5F
- J2, J3, J4, J5, J6: footprint TRS_JACK_WQP-PJ609B -> parts-for-kicad:TRS_JACK_WQP-PJ609B
- R25, R40, R43, R44, R46, R50, R51, R52, R53, R54, R59, R61, R64, R65, R68: footprint R0603 -> Resistor_SMD:R_0603_1608Metric
- SW1, SW2: footprint TOGGLE_SILK_PIP3 -> parts-for-kicad:TOGGLE_SILK_PIP3
- SW3: value SMT Mini Button -> PTH Mini Button; footprint TL3301SPF160QJ -> parts-for-kicad:TL1105SPF250Q; symbol Seed3-Pedal-DevKit-Converted-eagle-import:TAC_SWITCH_SMT -> parts-for-kicad:TAC_SWITCH_PTH
- U7: footprint MEM2061-01-188-00-A_GCT -> parts-for-kicad:MEM2061-01-188-00-A_GCT
- VR1, VR2, VR3: footprint 9MM_SNAP-IN_POT_SILK_PIP -> parts-for-kicad:9MM_SNAP-IN_POT_SILK_PIP
Connections:
- net +3V3: now also R28.2
- net +3V3_A: now also VR4.3, VR5.3, VR6.3
- net GND: now also J1.GND1 (PE), J1.GND2 (PE), J1.P2 (2), FSW_2.1 (S), LED1.1 (K), LED2.2 (K), SW4.3, SW4.4, SW6.2 (P), VR4.1, VR5.1, VR6.1
- net at R25.2: now also LED2.4 (GA)
- net at R43.2: now also LED1.2 (A)
- net at J1.P4 (4): now also R28.1
- net at J1.P5 (5): now also R29.2
- net at R44.2: now also LED2.3 (BA)
- net at R40.2: now also LED2.1 (RA)
- net +5V renamed +5V_A
- net TAC_SW renamed TAC_SW1
- new net GPIO_FSW_2: FSW_2.2 (S)
- new net MIDI_RX: R29.1
- new net POT_4: VR4.2
- new net POT_5: VR5.2
- new net POT_6: VR6.2
- new net TAC_SW2: SW4.1, SW4.2
- new net TOG_3: SW6.1 (O)
Other:
- note added: "MIDI IN"
- note added: "MIDI OUT"
- note added: "MIDI THRU"
- note removed: "TODO: MIDI Thru"
- moved on the sheet: C34, C47, J1, J10, J11, J2, J3, J4, J5, J6, R43, R46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

Commit message: fully routed.
Parts:
- SW2: symbol Seed3-Pedal-DevKit-Converted-eagle-import:TOGGLE_ON-ON_PIP3 -> parts-for-kicad:TOGGLE_ON-ON_PIP3
Changed lines of the file:
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@@
 	)
 	(symbol
-		(lib_id "Seed3-Pedal-DevKit-Converted-eagle-import:TOGGLE_ON-ON_PIP3")
+		(lib_id "parts-for-kicad:TOGGLE_ON-ON_PIP3")
 		(at 40.64 99.06 270)
 		(unit 1)

Commit message: first round of gerbs.
Parts:
- LED2: footprint LED_THT:LED_D5.0mm-4_RGB -> LED_THT:LED_D5.0mm-4_RGB_Wide_Pins
- SW3, SW4: value PTH Mini Button -> SMT Mini Button; footprint parts-for-kicad:TL1105SPF250Q -> parts-for-kicad:TL3301SPF160QJ; symbol parts-for-kicad:TAC_SWITCH_PTH -> parts-for-kicad:TAC_SWITCH_SMT
Changed lines of the file:
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@@
 	)
 	(symbol
-		(lib_id "parts-for-kicad:TAC_SWITCH_PTH")
+		(lib_id "parts-for-kicad:TAC_SWITCH_SMT")
 		(at 205.74 99.06 0)
 		(unit 1)
@@
 			)
 		)
-		(property "Value" "PTH Mini Button"
+		(property "Value" "SMT Mini Button"
 			(at 198.12 90.17 0)
 			(effects
@@
 			)
 		)
-		(property "Footprint" "parts-for-kicad:TL1105SPF250Q"
+		(property "Footprint" "parts-for-kicad:TL3301SPF160QJ"
 			(at 205.74 99.06 0)
 			(effects
@@
 			)
 		)
-		(property "Footprint" "LED_THT:LED_D5.0mm-4_RGB"
+		(property "Footprint" "LED_THT:LED_D5.0mm-4_RGB_Wide_Pins"
 			(at 171.45 176.53 0)
 			(effects
@@
 	)
 	(symbol
-		(lib_id "parts-for-kicad:TAC_SWITCH_PTH")
+		(lib_id "parts-for-kicad:TAC_SWITCH_SMT")
 		(at 167.64 99.06 0)
 		(unit 1)
@@
 			)
 		)
-		(property "Value" "PTH Mini Button"
+		(property "Value" "SMT Mini Button"
 			(at 160.02 90.17 0)
 			(effects
@@
 			)
 		)
-		(property "Footprint" "parts-for-kicad:TL1105SPF250Q"
+		(property "Footprint" "parts-for-kicad:TL3301SPF160QJ"
 			(at 167.64 99.06 0)
 			(effects
