File: pcb/ES-Seed3-DevKit-Pedal-Rev1/ES-Seed3-DevKit-Pedal-Rev1.kicad_sch (KiCad schematic)
At the start: 0 parts

Commit message: renamed project and remade gerbers.
Other:
- sheet ES_Daisy_Seed2_DFM_EVAL_PEDAL_Rev5_1 renamed ES-Seed3-DevKit-Pedal-Rev1_1
- sheet ES_Daisy_Seed2_DFM_EVAL_PEDAL_Rev5_2 renamed ES-Seed3-DevKit-Pedal-Rev1_2
- sheet ES_Daisy_Seed2_DFM_EVAL_PEDAL_Rev5_3 renamed ES-Seed3-DevKit-Pedal-Rev1_3
- sheet ES_Daisy_Seed2_DFM_EVAL_PEDAL_Rev5_4 renamed ES-Seed3-DevKit-Pedal-Rev1_4
- sheet ES-Seed3-DevKit-Pedal-Rev1_1: file ES_Daisy_Seed2_DFM_EVAL_PEDAL_Rev5_1.kicad_sch -> ES-Seed3-DevKit-Pedal-Rev1_1.kicad_sch
- sheet ES-Seed3-DevKit-Pedal-Rev1_2: file ES_Daisy_Seed2_DFM_EVAL_PEDAL_Rev5_2.kicad_sch -> ES-Seed3-DevKit-Pedal-Rev1_2.kicad_sch
- sheet ES-Seed3-DevKit-Pedal-Rev1_3: file ES_Daisy_Seed2_DFM_EVAL_PEDAL_Rev5_3.kicad_sch -> ES-Seed3-DevKit-Pedal-Rev1_3.kicad_sch
- sheet ES-Seed3-DevKit-Pedal-Rev1_4: file ES_Daisy_Seed2_DFM_EVAL_PEDAL_Rev5_4.kicad_sch -> ES-Seed3-DevKit-Pedal-Rev1_4.kicad_sch
Changed lines of the file:
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@@
 			(color 0 0 0 0.0000)
 		)
-		(property "Sheetname" "ES_Daisy_Seed2_DFM_EVAL_PEDAL_Rev5_2"
+		(property "Sheetname" "ES-Seed3-DevKit-Pedal-Rev1_2"
 			(at 76.2 24.6884 0)
 			(effects
@@
 			)
 		)
-		(property "Sheetfile" "ES_Daisy_Seed2_DFM_EVAL_PEDAL_Rev5_2.kicad_sch"
+		(property "Sheetfile" "ES-Seed3-DevKit-Pedal-Rev1_2.kicad_sch"
 			(at 76.2 29.7946 0)
 			(effects
@@
 		)
 		(instances
-			(project "Seed3-Pedal-DevKit-Converted"
+			(project "ES-Seed3-DevKit-Pedal-Rev1"
 				(path "/19edde5c-efb5-4a72-a9f3-fb5a3c99bba0"
 					(page "2")
@@
 			(color 0 0 0 0.0000)
 		)
-		(property "Sheetname" "ES_Daisy_Seed2_DFM_EVAL_PEDAL_Rev5_4"
+		(property "Sheetname" "ES-Seed3-DevKit-Pedal-Rev1_4"
 			(at 177.8 24.6884 0)
 			(effects
@@
 			)
 		)
-		(property "Sheetfile" "ES_Daisy_Seed2_DFM_EVAL_PEDAL_Rev5_4.kicad_sch"
+		(property "Sheetfile" "ES-Seed3-DevKit-Pedal-Rev1_4.kicad_sch"
 			(at 177.8 29.7946 0)
 			(effects
@@
 		)
 		(instances
-			(project "Seed3-Pedal-DevKit-Converted"
+			(project "ES-Seed3-DevKit-Pedal-Rev1"
 				(path "/19edde5c-efb5-4a72-a9f3-fb5a3c99bba0"
 					(page "4")
@@
 			(color 0 0 0 0.0000)
 		)
-		(property "Sheetname" "ES_Daisy_Seed2_DFM_EVAL_PEDAL_Rev5_3"
+		(property "Sheetname" "ES-Seed3-DevKit-Pedal-Rev1_3"
 			(at 127 24.6884 0)
 			(effects
@@
 			)
 		)
-		(property "Sheetfile" "ES_Daisy_Seed2_DFM_EVAL_PEDAL_Rev5_3.kicad_sch"
+		(property "Sheetfile" "ES-Seed3-DevKit-Pedal-Rev1_3.kicad_sch"
 			(at 127 29.7946 0)
 			(effects
@@
 		)
 		(instances
-			(project "Seed3-Pedal-DevKit-Converted"
+			(project "ES-Seed3-DevKit-Pedal-Rev1"
 				(path "/19edde5c-efb5-4a72-a9f3-fb5a3c99bba0"
 					(page "3")
@@
 			(color 0 0 0 0.0000)
 		)
-		(property "Sheetname" "ES_Daisy_Seed2_DFM_EVAL_PEDAL_Rev5_1"
+		(property "Sheetname" "ES-Seed3-DevKit-Pedal-Rev1_1"
 			(at 25.4 24.6884 0)
 			(effects
@@
 			)
 		)
-		(property "Sheetfile" "ES_Daisy_Seed2_DFM_EVAL_PEDAL_Rev5_1.kicad_sch"
+		(property "Sheetfile" "ES-Seed3-DevKit-Pedal-Rev1_1.kicad_sch"
 			(at 25.4 29.7946 0)
 			(effects
@@
 		)
 		(instances
-			(project "Seed3-Pedal-DevKit-Converted"
+			(project "ES-Seed3-DevKit-Pedal-Rev1"
 				(path "/19edde5c-efb5-4a72-a9f3-fb5a3c99bba0"
 					(page "1")
