File: pcb/ES-Seed3-DevKit-Pedal-Rev1/ES-Seed3-DevKit-Pedal-Rev1.kicad_pcb (KiCad board)
At the start: 2 copper layers, 197 x 100 mm, 166 parts, among them J1 DIN_MIDI_5P, J10 DIN_MIDI_5P, J11 DIN_MIDI_5P, J2 JACK_TRS_SWITCHING, J3 JACK_TRS_SWITCHING, J4 JACK_TRS_SWITCHING, J5 JACK_TRS_SWITCHING, J6 JACK_TRS_SWITCHING, J8 Barrel_Jack_Switch, Q1 3904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

Commit message: smt buttons pth again, and about to swap sd card.
Parts:
- SW3, SW4: value SMT Mini Button -> PTH Mini Button; footprint parts-for-kicad:TL3301SPF160QJ -> parts-for-kicad:TL1105SPF250Q_SILK
- turned SW3 to 0 degrees
- turned SW4 to 0 degrees
Routing:
- net TAC_SW2: track 112.6 -> 115.6 mm
- net TAC_SW1: track 101.8 -> 104.7 mm
