File: pcb/ES-Seed3-DevKit-Pedal-Rev1/ES-Seed3-DevKit-Pedal-Rev1.kicad_pcb (KiCad board)
At the start: 2 copper layers, 197 x 100 mm, 166 parts, among them J1 DIN_MIDI_5P, J10 DIN_MIDI_5P, J11 DIN_MIDI_5P, J2 JACK_TRS_SWITCHING, J3 JACK_TRS_SWITCHING, J4 JACK_TRS_SWITCHING, J5 JACK_TRS_SWITCHING, J6 JACK_TRS_SWITCHING, J8 Barrel_Jack_Switch, Q1 3904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

Commit message: new sdcard , lot of routing changes, and new gerbers
Parts:
- U7: footprint parts-for-kicad:MEM2061-01-188-00-A_GCT -> TF-01A:TF-01A
- moved U7 2.48 mm to (58.3, 136.7)
- moved R1 2.33 mm to (62.5, 80.5)
- moved R2 2.33 mm to (62.5, 86.0)
- moved U14 2.33 mm to (64.0, 83.2)
- moved U4 2.33 mm to (55.2, 83.2)
- moved C36 2.20 mm to (56.0, 103.0)
- moved C41 2.20 mm to (56.0, 95.6)
- moved L2 2.20 mm to (65.4, 99.0)
- moved R62 2.20 mm to (64.0, 92.3)
- moved R63 2.20 mm to (65.9, 92.3)
- moved A1 1.92 mm to (52.8, 125.3)
- moved R50 1.92 mm to (57.8, 121.8)
- moved R51 1.92 mm to (55.2, 121.8)
- moved R52 1.92 mm to (65.5, 121.8)
- moved R53 1.92 mm to (63.0, 121.8)
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Routing:
- net +3V3: track 368.0 -> 358.4 mm, vias 9 -> 10
- net /ES-Seed3-DevKit-Pedal-Rev1_1/USB_OTG_HS_N: track 44.8 -> 37.5 mm
- net /ES-Seed3-DevKit-Pedal-Rev1_1/USB_OTG_HS_P: track 39.1 -> 43.4 mm
- net SDMMC_D3: track 17.6 -> 20.9 mm
- net SDMMC_D0: track 16.5 -> 19.1 mm
- net SDMMC_D2: track 18.8 -> 20.8 mm
- net MIDI_TX: track 198.1 -> 200.1 mm
- net MIDI_RX: track 208.6 -> 210.5 mm
- net LED_MONO_1: track 141.8 -> 143.8 mm
- net GPIO_FSW_2: track 146.3 -> 148.2 mm
- net TOG_3: track 61.0 -> 62.9 mm
- net TOG_1: track 36.3 -> 38.3 mm
- net POT_5: track 116.2 -> 118.1 mm
- net POT_4: track 95.9 -> 97.8 mm
- net POT_3: track 119.7 -> 121.6 mm
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