File: pcb/ES-Seed3-DevKit-Pedal-Rev1/ES-Seed3-DevKit-Pedal-Rev1.kicad_pcb (KiCad board)
At the start: 2 copper layers, 197 x 100 mm, 166 parts, among them J1 DIN_MIDI_5P, J10 DIN_MIDI_5P, J11 DIN_MIDI_5P, J2 JACK_TRS_SWITCHING, J3 JACK_TRS_SWITCHING, J4 JACK_TRS_SWITCHING, J5 JACK_TRS_SWITCHING, J6 JACK_TRS_SWITCHING, J8 Barrel_Jack_Switch, Q1 3904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

Commit message: updated gerbs with matte material for mask.
Other:
- board text added: "Dielectric 1"
- board text added: "Matte"
- board text removed: "3.3"
- board text removed: "Dielectric"
