File: pcb/ES-Seed3-DevKit-Pedal-Rev1/ES-Seed3-DevKit-Pedal-Rev1_2.kicad_sch (KiCad schematic)
At the start: 43 parts, among them J1 DIN_MIDI_5P, J10 DIN_MIDI_5P, J11 DIN_MIDI_5P, J2 JACK_TRS_SWITCHING, J3 JACK_TRS_SWITCHING, J4 JACK_TRS_SWITCHING, J5 JACK_TRS_SWITCHING, J6 JACK_TRS_SWITCHING, SW1 TOGGLE_ON_OFF_ON_PIP2, SW2 TOGGLE_ON-ON_PIP3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

Commit message: smt buttons pth again, and about to swap sd card.
Parts:
- SW3, SW4: value SMT Mini Button -> PTH Mini Button; footprint parts-for-kicad:TL3301SPF160QJ -> parts-for-kicad:TL1105SPF250Q_SILK; symbol parts-for-kicad:TAC_SWITCH_SMT -> parts-for-kicad:TAC_SWITCH_PTH_SILK
Changed lines of the file:
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@@
 	)
 	(symbol
-		(lib_id "parts-for-kicad:TAC_SWITCH_SMT")
+		(lib_id "parts-for-kicad:TAC_SWITCH_PTH_SILK")
 		(at 205.74 99.06 0)
 		(unit 1)
@@
 			)
 		)
-		(property "Value" "SMT Mini Button"
+		(property "Value" "PTH Mini Button"
 			(at 198.12 90.17 0)
 			(effects
@@
 			)
 		)
-		(property "Footprint" "parts-for-kicad:TL3301SPF160QJ"
+		(property "Footprint" "parts-for-kicad:TL1105SPF250Q_SILK"
 			(at 205.74 99.06 0)
 			(effects
@@
 	)
 	(symbol
-		(lib_id "parts-for-kicad:TAC_SWITCH_SMT")
+		(lib_id "parts-for-kicad:TAC_SWITCH_PTH_SILK")
 		(at 167.64 99.06 0)
 		(unit 1)
@@
 			)
 		)
-		(property "Value" "SMT Mini Button"
+		(property "Value" "PTH Mini Button"
 			(at 160.02 90.17 0)
 			(effects
@@
 			)
 		)
-		(property "Footprint" "parts-for-kicad:TL3301SPF160QJ"
+		(property "Footprint" "parts-for-kicad:TL1105SPF250Q_SILK"
 			(at 167.64 99.06 0)
 			(effects

Commit message: new sdcard , lot of routing changes, and new gerbers
Parts:
- U7: footprint parts-for-kicad:MEM2061-01-188-00-A_GCT -> TF-01A:TF-01A; symbol Seed3-Pedal-DevKit-Converted-eagle-import:MICRO_SD_CARD -> TF-01A:TF-01A; Availability (none) -> Not in stock; Check_prices (none) -> https://www.snapeda.com/parts/TF-01A/HRO+Electronics+Co.%25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; Description_1 (none) -> Standard Card Edge Connectors; MF (none) -> HRO Electronics Co., Ltd.; MP (none) -> TF-01A; Package (none) -> Package; Price (none) -> None; SnapEDA_Link (none) -> https://www.snapeda.com/parts/TF-01A/HRO+Electronics+Co.%25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
Connections:
- net +3V3: now also U7.4 (VDD); no longer U7.P4 (VCC)
- net GND: now also U7.6 (VSS), U7.MP1 (SHIELD), U7.MP2 (SHIELD), U7.MP3 (SHIELD), U7.MP4 (SHIELD); no longer U7.11 (SHIELD@2), U7.12 (SHIELD@1), U7.P6 (GND)
- net SDMMC_CK: now also U7.5 (CLK); no longer U7.P5 (SCK)
- net SDMMC_CMD: now also U7.3 (CMD); no longer U7.P3 (CMD/DI)
- net SDMMC_D0: now also U7.7 (DAT0); no longer U7.P7 (D0/DO)
- net SDMMC_D1: now also U7.8 (DAT1); no longer U7.P8 (D1/RSV)
- net SDMMC_D2: now also U7.1 (DAT2); no longer U7.P1 (D2/NC)
- net SDMMC_D3: now also U7.2 (CD/DAT3); no longer U7.P2 (D3/CS)
Other:
- moved on the sheet: LED1, LED2, R25, R40, R43, R44, R50, R51, R52, R53, R54
