File: pcb/ES-Seed3-DevKit-Pedal-Rev2/ES-Seed3-DevKit-Pedal-Rev2.kicad_pcb (KiCad board)
At the start: 2 copper layers, 197 x 100 mm, 159 parts, among them J1 DIN_MIDI_5P, J10 DIN_MIDI_5P, J11 DIN_MIDI_5P, J2 JACK_TRS_SWITCHING, J3 JACK_TRS_SWITCHING, J4 JACK_TRS_SWITCHING, J5 JACK_TRS_SWITCHING, J6 JACK_TRS_SWITCHING, J7 USB4110GFA, J8 Barrel_Jack_Switch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

Commit message: I think schematic is done, board is updated -- needs layout and final routing.
Parts:
- removed D3, D4: 1N4148, Diode_SMD:D_SOD-323
- removed Q1, Q5: 3904, Package_TO_SOT_SMD:SOT-23
- removed R23, R24: 2K, Resistor_SMD:R_0603_1608Metric
- removed U5, U6: G6K-2F-Y-TR DC3, PCB_PCB_relays_2025-01-13:RELAY-SMD_G6K-2F-Y
- R10: value 2K -> 10K
- R9: value 2K -> 0R
- moved R10 97.6 mm to (36.8, 113.0), turned to 0 degrees
- moved R9 96.8 mm to (36.8, 110.5)
Connections:
- net /Audio I/O/ADC_EXPRESSION_PRE renamed /Audio IO/ADC_EXPRESSION_PRE
- A1 pad 12: /Daisy/GPIO_RELAY_L -> unconnected-(A1-I2C1_SCL-Pad12)
- A1 pad 13: /Daisy/GPIO_RELAY_R -> unconnected-(A1-I2C1_SDA-Pad13)
- C29 pad 2: AUDIO_BUFF_LEFT -> AUDIO_IN_LEFT
- C42 pad 1: AUDIO_DSP_LEFT -> AUDIO_OUT_LEFT
- C6 pad 1: AUDIO_DSP_RIGHT -> AUDIO_OUT_RIGHT
- C7 pad 2: AUDIO_BUFF_RIGHT -> AUDIO_IN_RIGHT
- R10 pad 1: Net-(Q1-B) -> +9V_A
- R10 pad 2: /Daisy/GPIO_RELAY_L -> Net-(U1A-+)
- R14 pad 1: AUDIO_DSP_RIGHT -> AUDIO_OUT_RIGHT
- R15 pad 2: +5V_A -> /Audio IO/AREF_AUDIO_IN_BIAS
- R5 pad 1: /Audio I/O/AREF_AUDIO_IN_BIAS -> /Audio IO/AREF_AUDIO_IN_BIAS
- R7 pad 2: +5V_A -> /Audio IO/AREF_AUDIO_IN_BIAS
- R77 pad 1: AUDIO_DSP_LEFT -> AUDIO_OUT_LEFT
- R9 pad 1: GND -> +5V_A
- R9 pad 2: Net-(Q1-B) -> Net-(U1A-+)
- U1 pad 1: /Audio I/O/AREF_AUDIO_IN_BIAS -> /Audio IO/AREF_AUDIO_IN_BIAS
- U1 pad 2: /Audio I/O/AREF_AUDIO_IN_BIAS -> /Audio IO/AREF_AUDIO_IN_BIAS
- U10 pad 3: +5V_A -> /Audio IO/AREF_AUDIO_IN_BIAS
- U10 pad 5: +5V_A -> /Audio IO/AREF_AUDIO_IN_BIAS
- U3 pad 5: /Audio I/O/AREF_AUDIO_IN_BIAS -> /Audio IO/AREF_AUDIO_IN_BIAS
- U9 pad 5: /Audio I/O/AREF_AUDIO_IN_BIAS -> /Audio IO/AREF_AUDIO_IN_BIAS
Routing:
- net unconnected-(A1-I2C1_SCL-Pad12): track 0.00 -> 93.9 mm, vias 0 -> 2
- net /Daisy/GPIO_RELAY_L: track 93.9 -> 0.00 mm, vias 2 -> 0
- net AUDIO_OUT_LEFT: track 74.2 -> 138.3 mm, vias 3 -> 5
- net AUDIO_DSP_LEFT: track 64.1 -> 0.00 mm, vias 2 -> 0
- net unconnected-(A1-I2C1_SDA-Pad13): track 0.00 -> 61.3 mm, vias 0 -> 2
- net /Daisy/GPIO_RELAY_R: track 61.3 -> 0.00 mm, vias 2 -> 0
- net AUDIO_DSP_RIGHT: track 55.7 -> 0.00 mm
- net AUDIO_OUT_RIGHT: track 64.9 -> 120.6 mm
- net /Audio IO/AREF_AUDIO_IN_BIAS: track 0.00 -> 54.7 mm, vias 0 -> 3
- net /Audio I/O/AREF_AUDIO_IN_BIAS: track 54.7 -> 0.00 mm, vias 3 -> 0
- net (no net): track 3.40 -> 25.1 mm
- net AUDIO_IN_LEFT: track 15.6 -> 34.4 mm
- net AUDIO_BUFF_LEFT: track 18.9 -> 0.00 mm
- net AUDIO_IN_RIGHT: track 15.6 -> 33.4 mm
- net AUDIO_BUFF_RIGHT: track 17.8 -> 0.00 mm
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
Commit message: board is done -- working on prod mat generation, and then reviewing
Parts:
- LOGO1: footprint parts-for-kicad:OSHW-LOGO-L_TEXT -> Symbol:OSHW-Logo2_14.6x12mm_SilkScreen
- moved R10 61.4 mm to (96.8, 100.0), turned to -90 degrees
- moved R9 60.4 mm to (96.8, 103.1), turned to 90 degrees
- moved C40 3.21 mm to (188.3, 86.2), turned to -90 degrees
- moved U2 2.80 mm to (191.1, 84.3), turned to -90 degrees
- moved LOGO1 1.95 mm to (134.0, 126.0)
- moved R55 0.70 mm to (166.8, 77.1)
- moved R48 0.70 mm to (175.6, 77.1)
- moved R57 0.30 mm to (189.5, 79.0), turned to -90 degrees
Routing:
- net unconnected-(A1-I2C1_SCL-Pad12): track 93.9 -> 0.00 mm, vias 2 -> 0
- net +3V3: track 358.4 -> 289.3 mm, vias 10 -> 4
- net /Audio IO/AREF_AUDIO_IN_BIAS: track 54.7 -> 118.8 mm, vias 3 -> 8
- net unconnected-(A1-I2C1_SDA-Pad13): track 61.3 -> 0.00 mm, vias 2 -> 0
- net +9V_A: track 138.1 -> 196.8 mm, vias 7 -> 9
- net AUDIO_OUT_LEFT: track 138.3 -> 86.4 mm, vias 5 -> 2
- net +5V_A: track 204.0 -> 171.9 mm, vias 5 -> 3
- net (no net): track 25.1 -> 0.00 mm
- net /Daisy/+5V_USB: track 2.12 -> 19.2 mm, vias 0 -> 2
- net Net-(D5-A): track 26.3 -> 11.5 mm
- net DSY_VIN: track 1.69 -> 13.6 mm
- net Net-(C41-Pad1): track 0.00 -> 7.90 mm
- net /Daisy/USB_IN_N: track 3.90 -> 10.6 mm, vias 0 -> 2
- net AUDIO_IN_LEFT: track 34.4 -> 28.2 mm
- net /Daisy/USB_IN_P: track 3.73 -> 9.69 mm
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Other:
- board text added: "Rev2"
- board text removed: "Rev1"

Commit message: updated board with requested changes, and remade prod.
Parts:
- SW1, SW2, SW6: footprint parts-for-kicad:TOGGLE_SILK_PIP3 -> parts-for-kicad:TOGGLE_SILK_PIP
- VR1, VR2, VR3, VR4, VR5, VR6: footprint parts-for-kicad:9MM_SNAP-IN_POT_SILK_PIP -> parts-for-kicad:9MM_SNAP-IN_POT_SILK
