File: pcb/ES-Seed3-DevKit-Pedal-Rev3/ES-Seed3-DevKit-Pedal-Rev1_4.kicad_sch (KiCad schematic)
At the start: 31 parts, among them J8 Barrel_Jack_Switch, U2 LP2985-5.0

Commit message: first review/prod folders after making all changes.
Connections:
- no-connect marks 0 -> 1
