File: pcb/ES-Seed3-DevKit-Pedal-Rev3/ES-Seed3-DevKit-Pedal-Rev1_2.kicad_sch (KiCad schematic)
At the start: 43 parts, among them J1 DIN_MIDI_5P, J10 DIN_MIDI_5P, J11 DIN_MIDI_5P, J2 JACK_TRS_SWITCHING, J3 JACK_TRS_SWITCHING, J4 JACK_TRS_SWITCHING, J5 JACK_TRS_SWITCHING, J6 JACK_TRS_SWITCHING, SW1 TOGGLE_ON_OFF_ON_PIP2, SW2 TOGGLE_ON-ON_PIP3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

Commit message: first review/prod folders after making all changes.
Parts:
- J2, J3, J4, J5, J6: symbol Seed3-Pedal-DevKit-Converted-eagle-import:JACK_TRS_SWITCHING -> Connector_Audio:AudioJack3_Switch
- VR1, VR2, VR3, VR4, VR5, VR6: value P-10K-B-R-PIP -> P-10K-B-R
Connections:
- net AUDIO_IN_LEFT: now also J2.T; no longer J2.2 (TIP)
- net AUDIO_IN_RIGHT: now also J4.T; no longer J4.2 (TIP)
- net AUDIO_OUT_LEFT: now also J3.T; no longer J3.2 (TIP)
- net AUDIO_OUT_RIGHT: now also J5.T; no longer J5.2 (TIP)
- net EXPRESSION_IN_EXT: now also J6.T; no longer J6.2 (TIP)
- net GND: now also J2.S, J3.S, J4.S, J5.S, J6.S; no longer J2.1 (SLEEVE), J3.1 (SLEEVE), J4.1 (SLEEVE), J5.1 (SLEEVE), J6.1 (SLEEVE)
- net SDMMC_DETECT: now reaches U7.CD1 (CD)
- net at R46.1: now also J6.R; no longer J6.3 (RING)
- net at R68.2: now also J6.TN; no longer J6.5 (TIP_SW)
- net at R64.2: now also J2.TN; no longer J2.5 (TIP_SW)
- net at R65.2: now also J4.TN; no longer J4.5 (TIP_SW)
- no-connect marks 0 -> 24
Other:
- moved on the sheet: R46, R64, R65, R68

Commit message: prod mats with last bits of silk adjustment.
Parts:
- renumbered SW6 to SW5
Connections:
- net TAC_SW1 renamed TAC_SW4
- net TAC_SW2 renamed TAC_SW5
- net TOG_1 renamed TOG_SW2
- net TOG_2_A renamed TOG_SW1_A
- net TOG_2_B renamed TOG_SW1_B
- net TOG_3 renamed TOG_SW3
Changed lines of the file:
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@@
 		)
 	)
-	(global_label "TAC_SW2"
+	(global_label "TAC_SW5"
 		(shape bidirectional)
 		(at 195.58 99.06 180)
@@
 		)
 	)
-	(global_label "TOG_2_A"
+	(global_label "TOG_SW1_A"
 		(shape bidirectional)
 		(at 86.36 96.52 0)
@@
 		)
 		(property "Intersheetrefs" "${INTERSHEET_REFS}"
-			(at 98.0197 96.52 0)
+			(at 100.6274 96.52 0)
 			(effects
 				(font
@@
 		)
 	)
-	(global_label "TOG_3"
+	(global_label "TOG_SW3"
 		(shape bidirectional)
 		(at 49.53 76.2 0)
@@
 		)
 		(property "Intersheetrefs" "${INTERSHEET_REFS}"
-			(at 59.1746 76.2 0)
+			(at 61.7823 76.2 0)
 			(effects
 				(font
@@
 		)
 	)
-	(global_label "TOG_2_B"
+	(global_label "TOG_SW1_B"
 		(shape bidirectional)
 		(at 86.36 101.6 0)
@@
 		)
 		(property "Intersheetrefs" "${INTERSHEET_REFS}"
-			(at 98.1975 101.6 0)
+			(at 100.8052 101.6 0)
 			(effects
 				(font
@@
 		)
 	)
-	(global_label "TAC_SW1"
+	(global_label "TAC_SW4"
 		(shape bidirectional)
 		(at 157.48 99.06 180)
@@
 		)
 	)
-	(global_label "TOG_1"
+	(global_label "TOG_SW2"
 		(shape bidirectional)
 		(at 48.26 96.52 0)
@@
 		)
 		(property "Intersheetrefs" "${INTERSHEET_REFS}"
-			(at 57.9046 96.52 0)
+			(at 60.5123 96.52 0)
 			(effects
 				(font
@@
 		(on_board yes)
 		(dnp no)
-		(property "Reference" "SW6"
+		(property "Reference" "SW5"
 			(at 203.2 92.71 0)
 			(effects
@@
 			(project "ES-Seed3-DevKit-Pedal-Rev1"
 				(path "/19edde5c-efb5-4a72-a9f3-fb5a3c99bba0/0fd2c796-fc28-4dbb-a19a-be32e6f577a0"
-					(reference "SW6")
+					(reference "SW5")
 					(unit 1)
 				)
