File: pcb/ES-Seed3-DevKit-Pedal-Rev3/ES-Seed3-DevKit-Pedal-Rev1_3.kicad_sch (KiCad schematic)
At the start: 60 parts, among them U1 MCP6002-xSN, U10 OPA1652, U3 OPA1652, U9 OPA1652

Commit message: fixed QR code to be correct destination link, and removed DNIs.
Parts:
- removed R56: 10K, Resistor_SMD:R_0603_1608Metric, symbol Seed3-Pedal-DevKit-Converted-eagle-import:Electrosmith-Passives_R-US_R0603
- removed R9: 0R, Resistor_SMD:R_0603_1608Metric, symbol Seed3-Pedal-DevKit-Converted-eagle-import:Electrosmith-Passives_R-US_R0603
